File: switch_matrix.kicad_sch (KiCad schematic)
At the start: 111 parts, among them Q1 PMOS, SW1 MX_SW_solder, SW10 MX_SW_solder, SW11 MX_SW_solder, SW12 MX_SW_solder, SW13 MX_SW_solder, SW14 MX_SW_solder, SW15 MX_SW_solder, SW16 MX_SW_solder, SW17 MX_SW_solder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

Commit message: Aug202023-7:30pm
Parts:
- added S7: MX_stab, PCM_marbastlib-mx:STAB_MX_P_7u, symbol marbastlib-mx:MX_stab

Commit message: Refactored to use RP2040
Connections:
- net at SW49.2: now also D41.2 (A), SW41.2
- net at D43.2 (A), SW43.2: now also SW51.2
- net at D42.2 (A), SW42.2: now also SW50.2
